File: CH32V003/Schematics/MiniMastermind/MiniMastermind.kicad_sch (KiCad schematic)
At the start: 28 parts, among them J1 Conn_01x06, J2 USB_C_Receptacle, SW1 SW_Push_45deg, SW2 SW_Push_45deg, SW3 SW_Push_45deg, SW4 SW_Push_45deg, SW5 Reset, SW6 Boot, SW7 ChKeys, U1 CH32X033F8P6

Commit message: Started mini mastermind
Parts:
- removed C1: 4.7uF, Capacitor_SMD:C_0805_2012Metric, symbol Device:C_Small
- removed C2, C5 (x2), C7: 100nF, Capacitor_SMD:C_0805_2012Metric, symbol Device:C_Small
- removed D5: WS2812B, UL_LED:SK6812SIDE-A-RVS, symbol LED:WS2812B
- removed D6, D7: LED_Small, LED_SMD:LED_0805_2012Metric, symbol Device:LED_Small
- removed J1: Conn_01x06, Connector_PinHeader_2.54mm:PinHeader_1x06_P2.54mm_Vertical, symbol Connector_Generic:Conn_01x06
- removed J2: USB_C_Receptacle, BadgePiratesFootprint:USB_C_Receptical-Jing, symbol Connector:USB_C_Receptacle
- removed SW2: SW_Push_45deg, Button_Switch_Keyboard:SW_Cherry_MX_1.00u_PCB, symbol Switch:SW_Push_45deg
- removed SW5: Reset, UL_Buttons:TS-1185-C-A-B-B, symbol Switch:SW_Push
- removed SW6: Boot, UL_Buttons:TS-1185-C-A-B-B, symbol Switch:SW_Push
- removed SW7: ChKeys, UL_Buttons:TS-1185-C-A-B-B, symbol Switch:SW_Push
- removed U1: CH32X033F8P6, Package_SO:TSSOP-20_4.4x6.5mm_P0.65mm, symbol ICs:CH32X033F8P6
- added C8: 10u, Capacitor_SMD:C_0805_2012Metric, symbol Device:C_Small
- added H1, H2, H3, H4: MountingHole, MountingHole:MountingHole_2.2mm_M2, symbol Mechanical:MountingHole
- added J1: Prog, Connector_PinHeader_2.54mm:PinHeader_1x03_P2.54mm_Vertical, symbol Connector_Generic:Conn_01x03
- added J3: OledDisplay, Connector_PinHeader_2.54mm:PinHeader_1x04_P2.54mm_Vertical, symbol Connector_Generic:Conn_01x04
- added J4: USB_C_Receptacle, UL_USB:USB_C_Receptical-Jing, symbol Connector:USB_C_Receptacle
- added J5: Conn_01x02, Connector_PinHeader_2.54mm:PinHeader_1x02_P2.54mm_Vertical, symbol Connector_Generic:Conn_01x02
- added JP1: JOpen, Jumper:SolderJumper-2_P1.3mm_Open_TrianglePad1.0x1.5mm, symbol Jumper:Jumper_2_Open
- added JP2: JClosed, Jumper:SolderJumper-2_P1.3mm_Bridged_Pad1.0x1.5mm, symbol Jumper:Jumper_2_Bridged
- added JP3: Jumper_2_Open, Jumper:SolderJumper-2_P1.3mm_Open_TrianglePad1.0x1.5mm, symbol Jumper:Jumper_2_Open
- added JP4: Jumper_2_Bridged, Jumper:SolderJumper-2_P1.3mm_Bridged_Pad1.0x1.5mm, symbol Jumper:Jumper_2_Bridged
- added SW2: Rotary_Encoder_Switch, cafebabe:EC11L1524E03_Rotary_Encoder, symbol Device:Rotary_Encoder_Switch
- added SW5: SW_Push_45deg, Button_Switch_Keyboard:SW_Cherry_MX_1.00u_PCB, symbol Switch:SW_Push_45deg
- added U1: TLV1117-33, Package_TO_SOT_SMD:SOT-223-3_TabPin2, symbol Regulator_Linear:TLV1117-33
- added U2: CH32V003F4P6, Package_SO:TSSOP-20_4.4x6.5mm_P0.65mm, symbol WCH:CH32V003F4P6
- C6: value 100nF -> 10u
- D1, D2, D3, D4: footprint UL_LED:SK6812SIDE-A-RVS -> UL_LED:SK6812-E_Reverse
- R1: value 4k7 -> 1.5k
- RN2: value R_Pack04 -> 5.1k
Connections:
- net +5V: now also C6.1, J4.A4 (VBUS), J4.A9 (VBUS), J4.B4 (VBUS), J4.B9 (VBUS), U1.3 (VI); no longer C3.2, C4.2, C6.2, R1.1, RN2.1 (R1.1), RN2.2 (R2.1)
- net D+: now also J4.A6 (D+), J4.B6 (D+), U2.19 (PD2)
- net D-: now also R1.2, J4.A7 (D-), J4.B7 (D-), U2.20 (PD3)
- net PA1: now also SW5.1, U2.5 (PA1); no longer SW3.1
- net PA2: now also D1.1 (DIN), U2.6 (PA2)
- net PC3: now also J5.2 (Pin_2), U2.13 (PC3); no longer D1.1 (DIN)
- net VSS: now also C3.2, C6.2, C8.2, J1.3 (Pin_3), J4.A1 (GND), J4.A12 (GND), J4.B1 (GND), J4.B12 (GND), J4.S1 (SHIELD), JP2.1 (A), JP3.1 (A), SW2.C, SW2.S1, SW5.2, U1.1 (GND), U2.7 (VSS); no longer C3.1, C6.1
- net at RN2.7 (R2.2): no longer RN2.8 (R1.2)
- net VCC: now reaches RN2.5 (R4.2), RN2.6 (R3.2)
- net VCC: now also C8.1, J1.1 (Pin_1), JP1.1 (A), JP4.2 (B), U1.2 (VO), U2.9 (VCC)
- net at RN1.5 (R4.2): now also J4.B5 (CC2)
- net at RN1.6 (R3.2): now also J4.A5 (CC1)
- net PA0 renamed PD7
- net PD7: now also U2.4 (PD7)
- net PA3 renamed PD5
- net PD5: now also U2.2 (PD5)
- net PA9 renamed SCL
- net SCL: now also J3.2 (Pin_2), U2.12 (PC2), U2.15 (PC5); no longer RN2.4 (R4.1)
- new net: J3.3 (Pin_3), JP3.2 (B), JP4.1 (A)
- new net: J3.4 (Pin_4), JP1.2 (B), JP2.2 (B)
- new net DPU: R1.1, U2.1 (PD4)
- new net PC4: J5.1 (Pin_1), U2.14 (PC4)
- new net PD6: SW3.1, U2.3 (PD6)
- new net RotaryA: C3.1, SW2.B, U2.8 (PD0)
- new net RotaryB: C4.2, SW2.A, U2.10 (PC0)
- new net RotaryS: SW2.S2, U2.17 (PC7)
- new net SDA: J3.1 (Pin_1), RN2.4 (R4.1), U2.11 (PC1), U2.16 (PC6)
- new net SWIO: J1.2 (Pin_2), U2.18 (SWIO)
- no-connect marks 15 -> 12

Commit message: Ordering Master Mind
Parts:
- D1, D2, D3, D4: footprint UL_LED:SK6812-E_Reverse -> UL_LED:SK6812-E_FaceUp
Connections:
- net +5V: now also D1.1 (VDD), D2.1 (VDD), D3.1 (VDD), D4.1 (VDD); no longer D1.2 (VDD), D2.2 (VDD), D3.2 (VDD), D4.2 (VDD)
- net PA2: now also D1.4 (DIN); no longer D1.1 (DIN)
- net PC3: now also J5.1 (Pin_1); no longer J5.2 (Pin_2)
- net PC4: now also J5.2 (Pin_2); no longer J5.1 (Pin_1)
- net SCL: no longer U2.15 (PC5)
- net SDA: no longer U2.16 (PC6)
- net VSS: now also D1.3 (VSS), D2.3 (VSS), D3.3 (VSS), D4.3 (VSS); no longer D1.4 (VSS), D2.4 (VSS), D3.4 (VSS), D4.4 (VSS)
- new net: D3.2 (DOUT), D4.4 (DIN)
- new net: D2.2 (DOUT), D3.4 (DIN)
- new net: D1.2 (DOUT), D2.4 (DIN)
- no-connect marks 12 -> 14
