File: CH32V006/Quark006/Schematics/_autosave-Quark006.kicad_sch (KiCad schematic)
At the start: 26 parts, among them J1 ESP32_USB, J10 Conn_01x08, J11 Conn_01x03, J2 WCH_USB, J3 Conn_01x06, J4 Conn_01x02, J5 Conn_01x02, J6 Conn_01x01, J7 Conn_01x01, J8 Conn_01x01, J9 Conn_01x01, SW1 SW_SPST, U1 ESP32-S2-MINI-1U-N4, U2 CH32V003FxPx, U3 TLV1117-33

Commit message: 006 dev board done but for the tweaking
Parts:
- J11: footprint (none) -> Connector_PinHeader_2.54mm:PinHeader_1x03_P2.54mm_Vertical
Changed lines of the file:
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@@
 			)
 		)
-		(property "Footprint" ""
+		(property "Footprint" "Connector_PinHeader_2.54mm:PinHeader_1x03_P2.54mm_Vertical"
 			(at 243.84 111.76 0)
 			(effects
