File: CH32V006/Quark006/Schematics/Quark006.kicad_pcb (KiCad board)
At the start: 2 copper layers, 59 x 30 mm, 43 parts, among them J1 ESP32_USB, J10 Conn_01x08, J11 Conn_01x03, J2 WCH_USB, J3 Conn_01x06, J4 Conn_01x02, J5 Conn_01x02, J6 Conn_01x01, J7 Conn_01x01, J8 Conn_01x01, J9 Conn_01x01, SW1 SW_SPST, U1 ESP32-S2-MINI-1U-N4, U2 CH32V003FxPx, U3 TLV1117-33

Commit message: moar
Parts:
- removed J11: Conn_01x03, Connector_PinHeader_2.54mm:PinHeader_1x03_P2.54mm_Vertical
- added J12: Conn_01x04, Connector_PinHeader_2.54mm:PinHeader_1x04_P2.54mm_Vertical, F.Cu at (205.0, 55.0)
- added JP1: Jumper_2_Bridged, Jumper:SolderJumper-2_P1.3mm_Bridged_RoundedPad1.0x1.5mm, B.Cu at (204.6, 50.4)
- added kibuzzard-67AFB7F8: G***, kibuzzard-67AFB7F8, F.Cu at (201.2, 55.6)
- added kibuzzard-67B101C4: G***, kibuzzard-67B101C4, F.Cu at (203.4, 49.0)
- added kibuzzard-67B10245: G***, kibuzzard-67B10245, B.Cu at (200.4, 74.6)
- added kibuzzard-67B102C6: G***, kibuzzard-67B102C6, F.Cu at (200.0, 53.2)
- moved RN1 17.3 mm to (185.1, 51.4), turned to 0 degrees
Connections:
- U2 pad 18: SWIO -> SWIOa
Routing:
- net SWIOa: track 0.00 -> 20.9 mm, vias 0 -> 1
- net CC1: track 11.7 -> 30.1 mm
- net CC2: track 10.4 -> 26.7 mm
- net VCC: track 85.5 -> 77.2 mm, vias 5 -> 4
- net SWIO: track 22.5 -> 15.9 mm, vias 2 -> 1
- net Net-(J1-CC2): track 12.2 -> 6.41 mm
- net +5V: track 61.9 -> 58.6 mm
- net Net-(J1-CC1): track 11.0 -> 9.40 mm
